File: boardAttinyReflexos/_autosave-attinyReflexos.kicad_pcb (KiCad board)
At the start: 2 copper layers, 43.2 x 43.2 mm, 17 parts, among them J1 Conn_01x06_Female, J2 Conn_01x03_Female, SW1 SW_DPST_x2, SW2 SW_DIP_x01, U1 ATTINY85-20PU

Commit message: caixa en openscad
Other:
- board text added: "pataTiny 1.0"
- board text removed: "quicky 0.2"
Changed lines of the file:
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@@
   )
   (setup
-    (last_trace_width 0.4)
+    (last_trace_width 0.2)
     (user_trace_width 0.2)
     (user_trace_width 0.4)
@@
     (tags "mounting hole 3.2mm no annular m3")
     (attr virtual)
-    (fp_text reference REF** (at 0 -4.2) (layer F.SilkS)
+    (fp_text reference REF** (at 0 -4.2) (layer F.SilkS) hide
       (effects (font (size 1 1) (thickness 0.15)))
     )
@@
     (tags "mounting hole 3.2mm no annular m3")
     (attr virtual)
-    (fp_text reference REF** (at 0 -4.2) (layer F.SilkS)
+    (fp_text reference REF** (at 0 -4.2) (layer F.SilkS) hide
       (effects (font (size 1 1) (thickness 0.15)))
     )
@@
     (tags "mounting hole 3.2mm no annular m3")
     (attr virtual)
-    (fp_text reference REF** (at 0 -4.2) (layer F.SilkS)
+    (fp_text reference REF** (at 0 -4.2) (layer F.SilkS) hide
       (effects (font (size 1 1) (thickness 0.15)))
     )
@@
     (tags "mounting hole 3.2mm no annular m3")
     (attr virtual)
-    (fp_text reference REF** (at 0 -4.2) (layer F.SilkS)
+    (fp_text reference REF** (at 0 -4.2) (layer F.SilkS) hide
       (effects (font (size 1 1) (thickness 0.15)))
     )
@@
     (effects (font (size 1.5 1.5) (thickness 0.3)) (justify mirror))
   )
-  (gr_text "quicky 0.2" (at 148.59 130.81) (layer F.SilkS)
+  (gr_text "pataTiny 1.0" (at 148.59 130.81) (layer F.SilkS)
     (effects (font (size 1.5 1.5) (thickness 0.3)))
   )
