File: boardAttinyReflexos/attinyReflexos.sch (KiCad schematic (older format))
At the start: 13 parts, among them J1 Conn_01x06_Female, SW1 SW_DPST_x2, SW2 SW_DIP_x01, U1 ATTINY85-20PU

Commit message: corrixido erro
Connections:
- net at U1.2 (PB3(XTAL1/CLKI/OC1B/ADC3/PCINT3)): now also R1.1, SW1.1 (A); no longer R4.1
- net at J1.3 (Pin_3), U1.5 (PB0(MOSI/DI/SDA/AIN0/OC0A/OC1A/AREF/PCINT0)): now also R2.1; no longer R1.1, SW1.1 (A)
- net at J1.4 (Pin_4), U1.6 (PB1(MISO/DO/AIN1/OC0B/OC1A/PCINT1)): now also R3.1; no longer R2.1
- net at J1.5 (Pin_5), U1.7 (PB2(SCK/USCK/SCL/T0/INT0/ADC1/PCINT2)): now also R4.1; no longer R3.1
Other:
- moved on the sheet: D1, D2, D3, R1, R2, R3, R4, SW1A
Changed lines of the file:
@@
 L R R3
 U 1 1 59CAB571
-P 2300 3050
-F 0 "R3" V 2380 3050 50  0000 C CNN
-F 1 "100" V 2300 3050 50  0000 C CNN
-F 2 "Resistors_ThroughHole:R_Axial_DIN0207_L6.3mm_D2.5mm_P7.62mm_Horizontal" V 2230 3050 50  0001 C CNN
-F 3 "" H 2300 3050 50  0001 C CNN
-	1    2300 3050
+P 1700 3050
+F 0 "R3" V 1780 3050 50  0000 C CNN
+F 1 "100" V 1700 3050 50  0000 C CNN
+F 2 "Resistors_ThroughHole:R_Axial_DIN0207_L6.3mm_D2.5mm_P7.62mm_Horizontal" V 1630 3050 50  0001 C CNN
+F 3 "" H 1700 3050 50  0001 C CNN
+	1    1700 3050
 	1    0    0    -1
 $EndComp
@@
 L R R4
 U 1 1 59CAB662
-P 2650 3050
-F 0 "R4" V 2730 3050 50  0000 C CNN
-F 1 "100" V 2650 3050 50  0000 C CNN
-F 2 "Resistors_ThroughHole:R_Axial_DIN0207_L6.3mm_D2.5mm_P7.62mm_Horizontal" V 2580 3050 50  0001 C CNN
-F 3 "" H 2650 3050 50  0001 C CNN
-	1    2650 3050
+P 2100 3050
+F 0 "R4" V 2180 3050 50  0000 C CNN
+F 1 "100" V 2100 3050 50  0000 C CNN
+F 2 "Resistors_ThroughHole:R_Axial_DIN0207_L6.3mm_D2.5mm_P7.62mm_Horizontal" V 2030 3050 50  0001 C CNN
+F 3 "" H 2100 3050 50  0001 C CNN
+	1    2100 3050
 	1    0    0    -1
 $EndComp
@@
 L R R2
 U 1 1 59CAB6B1
-P 2000 3050
-F 0 "R2" V 2080 3050 50  0000 C CNN
-F 1 "100" V 2000 3050 50  0000 C CNN
-F 2 "Resistors_ThroughHole:R_Axial_DIN0207_L6.3mm_D2.5mm_P7.62mm_Horizontal" V 1930 3050 50  0001 C CNN
-F 3 "" H 2000 3050 50  0001 C CNN
-	1    2000 3050
+P 1250 3050
+F 0 "R2" V 1330 3050 50  0000 C CNN
+F 1 "100" V 1250 3050 50  0000 C CNN
+F 2 "Resistors_ThroughHole:R_Axial_DIN0207_L6.3mm_D2.5mm_P7.62mm_Horizontal" V 1180 3050 50  0001 C CNN
+F 3 "" H 1250 3050 50  0001 C CNN
+	1    1250 3050
 	1    0    0    -1
 $EndComp
@@
 L LED D2
 U 1 1 59CAB6CC
-P 2300 3450
-F 0 "D2" H 2300 3550 50  0000 C CNN
-F 1 "LED" H 2300 3350 50  0000 C CNN
-F 2 "LEDs:LED_D5.0mm" H 2300 3450 50  0001 C CNN
-F 3 "" H 2300 3450 50  0001 C CNN
-	1    2300 3450
+P 1700 3450
+F 0 "D2" H 1700 3550 50  0000 C CNN
+F 1 "LED" H 1700 3350 50  0000 C CNN
+F 2 "LEDs:LED_D5.0mm" H 1700 3450 50  0001 C CNN
+F 3 "" H 1700 3450 50  0001 C CNN
+	1    1700 3450
 	0    -1   -1   0
 $EndComp
@@
 L LED D1
 U 1 1 59CAB7D2
-P 2000 3450
-F 0 "D1" H 2000 3550 50  0000 C CNN
-F 1 "LED" H 2000 3350 50  0000 C CNN
-F 2 "LEDs:LED_D5.0mm" H 2000 3450 50  0001 C CNN
-F 3 "" H 2000 3450 50  0001 C CNN
-	1    2000 3450
+P 1250 3450
+F 0 "D1" H 1250 3550 50  0000 C CNN
+F 1 "LED" H 1250 3350 50  0000 C CNN
+F 2 "LEDs:LED_D5.0mm" H 1250 3450 50  0001 C CNN
+F 3 "" H 1250 3450 50  0001 C CNN
+	1    1250 3450
 	0    -1   -1   0
 $EndComp
@@
 L LED D3
 U 1 1 59CAB7FE
-P 2650 3450
-F 0 "D3" H 2650 3550 50  0000 C CNN
-F 1 "LED" H 2650 3350 50  0000 C CNN
-F 2 "LEDs:LED_D5.0mm" H 2650 3450 50  0001 C CNN
-F 3 "" H 2650 3450 50  0001 C CNN
-	1    2650 3450
+P 2100 3450
+F 0 "D3" H 2100 3550 50  0000 C CNN
+F 1 "LED" H 2100 3350 50  0000 C CNN
+F 2 "LEDs:LED_D5.0mm" H 2100 3450 50  0001 C CNN
+F 3 "" H 2100 3450 50  0001 C CNN
+	1    2100 3450
 	0    -1   -1   0
 $EndComp
@@
 L SW_DPST_x2 SW1
 U 1 1 59CAB9A7
-P 1600 2200
-F 0 "SW1" H 1600 2325 50  0000 C CNN
-F 1 "SW_DPST_x2" H 1600 2100 50  0000 C CNN
-F 2 "Buttons_Switches_ThroughHole:SW_PUSH_6mm_h5mm" H 1600 2200 50  0001 C CNN
-F 3 "" H 1600 2200 50  0001 C CNN
-	1    1600 2200
+P 2500 3850
+F 0 "SW1" H 2500 3975 50  0000 C CNN
+F 1 "SW_DPST_x2" H 2500 3750 50  0000 C CNN
+F 2 "Buttons_Switches_ThroughHole:SW_PUSH_6mm_h5mm" H 2500 3850 50  0001 C CNN
+F 3 "" H 2500 3850 50  0001 C CNN
+	1    2500 3850
 	0    -1   -1   0
 $EndComp
@@
 L GND #PWR01
 U 1 1 5A74B21D
-P 2000 3750
-F 0 "#PWR01" H 2000 3500 50  0001 C CNN
-F 1 "GND" H 2000 3600 50  0000 C CNN
-F 2 "" H 2000 3750 50  0001 C CNN
-F 3 "" H 2000 3750 50  0001 C CNN
-	1    2000 3750
+P 1250 3750
+F 0 "#PWR01" H 1250 3500 50  0001 C CNN
+F 1 "GND" H 1250 3600 50  0000 C CNN
+F 2 "" H 1250 3750 50  0001 C CNN
+F 3 "" H 1250 3750 50  0001 C CNN
+	1    1250 3750
 	1    0    0    -1
 $EndComp
@@
 L R R1
 U 1 1 5A74B427
-P 1600 3050
-F 0 "R1" V 1680 3050 50  0000 C CNN
-F 1 "10K" V 1600 3050 50  0000 C CNN
-F 2 "Resistors_ThroughHole:R_Axial_DIN0207_L6.3mm_D2.5mm_P7.62mm_Horizontal" V 1530 3050 50  0001 C CNN
-F 3 "" H 1600 3050 50  0001 C CNN
-	1    1600 3050
+P 2500 4700
+F 0 "R1" V 2580 4700 50  0000 C CNN
+F 1 "10K" V 2500 4700 50  0000 C CNN
+F 2 "Resistors_ThroughHole:R_Axial_DIN0207_L6.3mm_D2.5mm_P7.62mm_Horizontal" V 2430 4700 50  0001 C CNN
+F 3 "" H 2500 4700 50  0001 C CNN
+	1    2500 4700
 	1    0    0    -1
 $EndComp
@@
 L VCC #PWR02
 U 1 1 5A74B55B
-P 1600 1900
-F 0 "#PWR02" H 1600 1750 50  0001 C CNN
-F 1 "VCC" H 1600 2050 50  0000 C CNN
-F 2 "" H 1600 1900 50  0001 C CNN
-F 3 "" H 1600 1900 50  0001 C CNN
-	1    1600 1900
-	1    0    0    -1
-$EndComp
-Wire Wire Line
-	2650 3200 2650 3300
-Wire Wire Line
-	2300 3200 2300 3300
-Wire Wire Line
-	2000 3200 2000 3300
+P 2500 3550
+F 0 "#PWR02" H 2500 3400 50  0001 C CNN
+F 1 "VCC" H 2500 3700 50  0000 C CNN
+F 2 "" H 2500 3550 50  0001 C CNN
+F 3 "" H 2500 3550 50  0001 C CNN
+	1    2500 3550
+	1    0    0    -1
+$EndComp
+Wire Wire Line
+	2100 3200 2100 3300
+Wire Wire Line
+	1700 3200 1700 3300
+Wire Wire Line
+	1250 3200 1250 3300
 Wire Wire Line
 	6000 2600 6400 2600
@@
 Connection ~ 6200 3100
 Wire Wire Line
-	2650 2900 3300 2900
-Wire Wire Line
-	2000 2900 2000 2900
-Wire Wire Line
-	2300 2900 2300 2800
-Wire Wire Line
-	2300 2800 3300 2800
-Wire Wire Line
-	2000 2900 2000 2700
-Wire Wire Line
-	2000 2700 3300 2700
-Wire Wire Line
-	2650 3600 2650 3750
-Wire Wire Line
-	2300 3600 2300 3750
-Wire Wire Line
-	2000 3600 2000 3750
-Wire Wire Line
-	1600 3200 1600 3750
-Wire Wire Line
-	1600 1900 1600 2000
-Wire Wire Line
-	1600 2400 1600 2900
-Wire Wire Line
-	3300 2600 1600 2600
-Connection ~ 1600 2600
+	2100 3600 2100 3750
+Wire Wire Line
+	1700 3600 1700 3750
+Wire Wire Line
+	1250 3600 1250 3750
+Wire Wire Line
+	2500 4850 2500 5400
+Wire Wire Line
+	2500 3550 2500 3650
+Wire Wire Line
+	2500 4050 2500 4550
+Connection ~ 2500 4250
 $Comp
 L GND #PWR03
 U 1 1 5A74B1B1
-P 2650 3750
-F 0 "#PWR03" H 2650 3500 50  0001 C CNN
-F 1 "GND" H 2650 3600 50  0000 C CNN
-F 2 "" H 2650 3750 50  0001 C CNN
-F 3 "" H 2650 3750 50  0001 C CNN
-	1    2650 3750
+P 2100 3750
+F 0 "#PWR03" H 2100 3500 50  0001 C CNN
+F 1 "GND" H 2100 3600 50  0000 C CNN
+F 2 "" H 2100 3750 50  0001 C CNN
+F 3 "" H 2100 3750 50  0001 C CNN
+	1    2100 3750
 	1    0    0    -1
 $EndComp
@@
 L GND #PWR04
 U 1 1 5A74B1E4
-P 2300 3750
-F 0 "#PWR04" H 2300 3500 50  0001 C CNN
-F 1 "GND" H 2300 3600 50  0000 C CNN
-F 2 "" H 2300 3750 50  0001 C CNN
-F 3 "" H 2300 3750 50  0001 C CNN
-	1    2300 3750
+P 1700 3750
+F 0 "#PWR04" H 1700 3500 50  0001 C CNN
+F 1 "GND" H 1700 3600 50  0000 C CNN
+F 2 "" H 1700 3750 50  0001 C CNN
+F 3 "" H 1700 3750 50  0001 C CNN
+	1    1700 3750
 	1    0    0    -1
 $EndComp
@@
 L GND #PWR05
 U 1 1 5A74B35F
-P 1600 3750
-F 0 "#PWR05" H 1600 3500 50  0001 C CNN
-F 1 "GND" H 1600 3600 50  0000 C CNN
-F 2 "" H 1600 3750 50  0001 C CNN
-F 3 "" H 1600 3750 50  0001 C CNN
-	1    1600 3750
+P 2500 5400
+F 0 "#PWR05" H 2500 5150 50  0001 C CNN
+F 1 "GND" H 2500 5250 50  0000 C CNN
+F 2 "" H 2500 5400 50  0001 C CNN
+F 3 "" H 2500 5400 50  0001 C CNN
+	1    2500 5400
 	1    0    0    -1
 $EndComp
@@
 	6850 3800 3200 3800
 Wire Wire Line
-	3200 3800 3200 2600
-Connection ~ 3200 2600
-Wire Wire Line
 	6850 3900 3100 3900
-Wire Wire Line
-	3100 3900 3100 2700
 Connection ~ 3100 2700
 Wire Wire Line
 	6850 4000 3000 4000
-Wire Wire Line
-	3000 4000 3000 2800
 Connection ~ 3000 2800
 Wire Wire Line
@@
 	1    0    0    -1
 $EndComp
+Wire Wire Line
+	3000 4000 3000 2800
+Wire Wire Line
+	3100 3900 3100 2700
+Wire Wire Line
+	3200 3800 3200 2600
+Connection ~ 3200 2600
+Wire Wire Line
+	1250 2600 3300 2600
+Wire Wire Line
+	1700 2700 3300 2700
+Wire Wire Line
+	2100 2800 3300 2800
+Wire Wire Line
+	1250 2600 1250 2900
+Wire Wire Line
+	1700 2700 1700 2900
+Wire Wire Line
+	2100 2800 2100 2900
+Wire Wire Line
+	3300 2900 2850 2900
+Wire Wire Line
+	2850 2900 2850 4250
+Wire Wire Line
+	2850 4250 2500 4250
 $EndSCHEMATC

Commit message: big updates
Parts:
- removed C1: 10uF, Capacitors_ThroughHole:CP_Radial_D5.0mm_P2.50mm, symbol C_Small
- added J2: Conn_01x03_Female, Pin_Headers:Pin_Header_Angled_1x03_Pitch2.54mm, symbol Conn_01x03_Female
- D1, D2, D3: footprint LEDs:LED_D5.0mm -> LEDs:LED_D3.0mm
- R1, R2, R3, R4: footprint Resistors_ThroughHole:R_Axial_DIN0207_L6.3mm_D2.5mm_P7.62mm_Horizontal -> myfootprint:R_Axial_DIN0207_L6.3mm_D2.5mm_P7.62mm_Horizontal
- SW1: footprint Buttons_Switches_ThroughHole:SW_PUSH_6mm_h5mm -> myfootprint:SW_PUSH_6mm_H5mm
- SW2: footprint Choke_Toroid_ThroughHole:Choke_Toroid_horizontal_Diameter6mm_Amidon-T20 -> myfootprint:switchSlide
Connections:
- net GND: now also J2.1 (Pin_1)
- net VCC: now also J2.2 (Pin_2)
- net at U1.3 (PB4(XTAL2/CLKO/OC1B/ADC2/PCINT4)): now also J2.3 (Pin_3)
- no-connect marks 1 -> 0
Other:
- moved on the sheet: BT1
Changed lines of the file:
@@
 F 0 "R3" V 1780 3050 50  0000 C CNN
 F 1 "100" V 1700 3050 50  0000 C CNN
-F 2 "Resistors_ThroughHole:R_Axial_DIN0207_L6.3mm_D2.5mm_P7.62mm_Horizontal" V 1630 3050 50  0001 C CNN
+F 2 "myfootprint:R_Axial_DIN0207_L6.3mm_D2.5mm_P7.62mm_Horizontal" V 1630 3050 50  0001 C CNN
 F 3 "" H 1700 3050 50  0001 C CNN
 	1    1700 3050
@@
 F 0 "R4" V 2180 3050 50  0000 C CNN
 F 1 "100" V 2100 3050 50  0000 C CNN
-F 2 "Resistors_ThroughHole:R_Axial_DIN0207_L6.3mm_D2.5mm_P7.62mm_Horizontal" V 2030 3050 50  0001 C CNN
+F 2 "myfootprint:R_Axial_DIN0207_L6.3mm_D2.5mm_P7.62mm_Horizontal" V 2030 3050 50  0001 C CNN
 F 3 "" H 2100 3050 50  0001 C CNN
 	1    2100 3050
@@
 F 0 "R2" V 1330 3050 50  0000 C CNN
 F 1 "100" V 1250 3050 50  0000 C CNN
-F 2 "Resistors_ThroughHole:R_Axial_DIN0207_L6.3mm_D2.5mm_P7.62mm_Horizontal" V 1180 3050 50  0001 C CNN
+F 2 "myfootprint:R_Axial_DIN0207_L6.3mm_D2.5mm_P7.62mm_Horizontal" V 1180 3050 50  0001 C CNN
 F 3 "" H 1250 3050 50  0001 C CNN
 	1    1250 3050
@@
 F 0 "D2" H 1700 3550 50  0000 C CNN
 F 1 "LED" H 1700 3350 50  0000 C CNN
-F 2 "LEDs:LED_D5.0mm" H 1700 3450 50  0001 C CNN
+F 2 "LEDs:LED_D3.0mm" H 1700 3450 50  0001 C CNN
 F 3 "" H 1700 3450 50  0001 C CNN
 	1    1700 3450
@@
 F 0 "D1" H 1250 3550 50  0000 C CNN
 F 1 "LED" H 1250 3350 50  0000 C CNN
-F 2 "LEDs:LED_D5.0mm" H 1250 3450 50  0001 C CNN
+F 2 "LEDs:LED_D3.0mm" H 1250 3450 50  0001 C CNN
 F 3 "" H 1250 3450 50  0001 C CNN
 	1    1250 3450
@@
 F 0 "D3" H 2100 3550 50  0000 C CNN
 F 1 "LED" H 2100 3350 50  0000 C CNN
-F 2 "LEDs:LED_D5.0mm" H 2100 3450 50  0001 C CNN
+F 2 "LEDs:LED_D3.0mm" H 2100 3450 50  0001 C CNN
 F 3 "" H 2100 3450 50  0001 C CNN
 	1    2100 3450
@@
 F 0 "SW1" H 2500 3975 50  0000 C CNN
 F 1 "SW_DPST_x2" H 2500 3750 50  0000 C CNN
-F 2 "Buttons_Switches_ThroughHole:SW_PUSH_6mm_h5mm" H 2500 3850 50  0001 C CNN
+F 2 "myfootprint:SW_PUSH_6mm_H5mm" H 2500 3850 50  0001 C CNN
 F 3 "" H 2500 3850 50  0001 C CNN
 	1    2500 3850
@@
 L Battery_Cell BT1
 U 1 1 59D92230
-P 7200 2800
-F 0 "BT1" H 7300 2900 50  0000 L CNN
-F 1 "Battery_Cell" H 7300 2800 50  0000 L CNN
-F 2 "Battery_Holders:Keystone_103_1x20mm-CoinCell" V 7200 2860 50  0001 C CNN
-F 3 "" V 7200 2860 50  0001 C CNN
-	1    7200 2800
-	1    0    0    -1
-$EndComp
-$Comp
-L C_Small C1
-U 1 1 59D924A0
-P 6200 2850
-F 0 "C1" H 6210 2920 50  0000 L CNN
-F 1 "10uF" H 6210 2770 50  0000 L CNN
-F 2 "Capacitors_ThroughHole:CP_Radial_D5.0mm_P2.50mm" H 6200 2850 50  0001 C CNN
-F 3 "" H 6200 2850 50  0001 C CNN
-	1    6200 2850
+P 7200 2900
+F 0 "BT1" H 7300 3000 50  0000 L CNN
+F 1 "Battery_Cell" H 7300 2900 50  0000 L CNN
+F 2 "Battery_Holders:Keystone_103_1x20mm-CoinCell" V 7200 2960 50  0001 C CNN
+F 3 "" V 7200 2960 50  0001 C CNN
+	1    7200 2900
 	1    0    0    -1
 $EndComp
@@
 F 0 "R1" V 2580 4700 50  0000 C CNN
 F 1 "10K" V 2500 4700 50  0000 C CNN
-F 2 "Resistors_ThroughHole:R_Axial_DIN0207_L6.3mm_D2.5mm_P7.62mm_Horizontal" V 2430 4700 50  0001 C CNN
+F 2 "myfootprint:R_Axial_DIN0207_L6.3mm_D2.5mm_P7.62mm_Horizontal" V 2430 4700 50  0001 C CNN
 F 3 "" H 2500 4700 50  0001 C CNN
 	1    2500 4700
@@
 	1    0    0    -1
 $EndComp
-Wire Wire Line
-	2100 3200 2100 3300
-Wire Wire Line
-	1700 3200 1700 3300
-Wire Wire Line
-	1250 3200 1250 3300
-Wire Wire Line
-	6000 2600 6400 2600
-Wire Wire Line
-	7200 2600 7000 2600
-Wire Wire Line
-	7200 3100 7200 2900
-Wire Wire Line
-	6000 3100 7200 3100
-Wire Wire Line
-	6200 2500 6200 2750
-Connection ~ 6200 2600
-Wire Wire Line
-	6200 2950 6200 3200
-Connection ~ 6200 3100
-Wire Wire Line
-	2100 3600 2100 3750
-Wire Wire Line
-	1700 3600 1700 3750
-Wire Wire Line
-	1250 3600 1250 3750
-Wire Wire Line
-	2500 4850 2500 5400
-Wire Wire Line
-	2500 3550 2500 3650
-Wire Wire Line
-	2500 4050 2500 4550
-Connection ~ 2500 4250
 $Comp
 L GND #PWR03
@@
 L VCC #PWR06
 U 1 1 5A74BBC2
-P 6200 2500
-F 0 "#PWR06" H 6200 2350 50  0001 C CNN
-F 1 "VCC" H 6200 2650 50  0000 C CNN
-F 2 "" H 6200 2500 50  0001 C CNN
-F 3 "" H 6200 2500 50  0001 C CNN
-	1    6200 2500
+P 6250 2450
+F 0 "#PWR06" H 6250 2300 50  0001 C CNN
+F 1 "VCC" H 6250 2600 50  0000 C CNN
+F 2 "" H 6250 2450 50  0001 C CNN
+F 3 "" H 6250 2450 50  0001 C CNN
+	1    6250 2450
 	1    0    0    -1
 $EndComp
@@
 L GND #PWR07
 U 1 1 5A74BC27
-P 6200 3200
-F 0 "#PWR07" H 6200 2950 50  0001 C CNN
-F 1 "GND" H 6200 3050 50  0000 C CNN
-F 2 "" H 6200 3200 50  0001 C CNN
-F 3 "" H 6200 3200 50  0001 C CNN
-	1    6200 3200
+P 7200 3150
+F 0 "#PWR07" H 7200 2900 50  0001 C CNN
+F 1 "GND" H 7200 3000 50  0000 C CNN
+F 2 "" H 7200 3150 50  0001 C CNN
+F 3 "" H 7200 3150 50  0001 C CNN
+	1    7200 3150
 	1    0    0    -1
 $EndComp
@@
 L PWR_FLAG #FLG08
 U 1 1 5A74BF8B
-P 4250 4400
-F 0 "#FLG08" H 4250 4475 50  0001 C CNN
-F 1 "PWR_FLAG" H 4250 4550 50  0000 C CNN
-F 2 "" H 4250 4400 50  0001 C CNN
-F 3 "" H 4250 4400 50  0001 C CNN
-	1    4250 4400
+P 1300 4700
+F 0 "#FLG08" H 1300 4775 50  0001 C CNN
+F 1 "PWR_FLAG" H 1300 4850 50  0000 C CNN
+F 2 "" H 1300 4700 50  0001 C CNN
+F 3 "" H 1300 4700 50  0001 C CNN
+	1    1300 4700
 	1    0    0    -1
 $EndComp
@@
 L PWR_FLAG #FLG09
 U 1 1 5A74BFFF
-P 4800 4550
-F 0 "#FLG09" H 4800 4625 50  0001 C CNN
-F 1 "PWR_FLAG" H 4800 4700 50  0000 C CNN
-F 2 "" H 4800 4550 50  0001 C CNN
-F 3 "" H 4800 4550 50  0001 C CNN
-	1    4800 4550
+P 1850 4850
+F 0 "#FLG09" H 1850 4925 50  0001 C CNN
+F 1 "PWR_FLAG" H 1850 5000 50  0000 C CNN
+F 2 "" H 1850 4850 50  0001 C CNN
+F 3 "" H 1850 4850 50  0001 C CNN
+	1    1850 4850
 	-1   0    0    1
 $EndComp
@@
 L GND #PWR010
 U 1 1 5A74C035
-P 4250 4550
-F 0 "#PWR010" H 4250 4300 50  0001 C CNN
-F 1 "GND" H 4250 4400 50  0000 C CNN
-F 2 "" H 4250 4550 50  0001 C CNN
-F 3 "" H 4250 4550 50  0001 C CNN
-	1    4250 4550
+P 1300 4850
+F 0 "#PWR010" H 1300 4600 50  0001 C CNN
+F 1 "GND" H 1300 4700 50  0000 C CNN
+F 2 "" H 1300 4850 50  0001 C CNN
+F 3 "" H 1300 4850 50  0001 C CNN
+	1    1300 4850
 	1    0    0    -1
 $EndComp
@@
 L VCC #PWR011
 U 1 1 5A74C064
-P 4800 4400
-F 0 "#PWR011" H 4800 4250 50  0001 C CNN
-F 1 "VCC" H 4800 4550 50  0000 C CNN
-F 2 "" H 4800 4400 50  0001 C CNN
-F 3 "" H 4800 4400 50  0001 C CNN
-	1    4800 4400
-	1    0    0    -1
-$EndComp
-Wire Wire Line
-	4800 4400 4800 4550
-Wire Wire Line
-	4250 4400 4250 4550
+P 1850 4700
+F 0 "#PWR011" H 1850 4550 50  0001 C CNN
+F 1 "VCC" H 1850 4850 50  0000 C CNN
+F 2 "" H 1850 4700 50  0001 C CNN
+F 3 "" H 1850 4700 50  0001 C CNN
+	1    1850 4700
+	1    0    0    -1
+$EndComp
 $Comp
 L Conn_01x06_Female J1
@@
 	1    0    0    -1
 $EndComp
-Wire Wire Line
-	6850 3700 3300 3700
-Wire Wire Line
-	3300 3700 3300 3100
-Wire Wire Line
-	6850 3800 3200 3800
-Wire Wire Line
-	6850 3900 3100 3900
-Connection ~ 3100 2700
-Wire Wire Line
-	6850 4000 3000 4000
-Connection ~ 3000 2800
-Wire Wire Line
-	6850 3600 6700 3600
-Wire Wire Line
-	6850 4100 6050 4100
-Wire Wire Line
-	6700 3600 6700 3100
-Connection ~ 6700 3100
-Wire Wire Line
-	6050 4100 6050 2600
-Connection ~ 6050 2600
-NoConn ~ 3300 3000
 $Comp
 L SW_DIP_x01 SW2
@@
 F 0 "SW2" H 6700 2750 50  0000 C CNN
 F 1 "SW_DIP_x01" H 6700 2450 50  0000 C CNN
-F 2 "Choke_Toroid_ThroughHole:Choke_Toroid_horizontal_Diameter6mm_Amidon-T20" H 6700 2600 50  0001 C CNN
+F 2 "myfootprint:switchSlide" H 6700 2600 50  0001 C CNN
 F 3 "" H 6700 2600 50  0001 C CNN
 	1    6700 2600
 	1    0    0    -1
 $EndComp
+$Comp
+L Conn_01x03_Female J2
+U 1 1 5B393E6D
+P 3800 2000
+F 0 "J2" H 3800 2200 50  0000 C CNN
+F 1 "Conn_01x03_Female" H 3800 1800 50  0000 C CNN
+F 2 "Pin_Headers:Pin_Header_Angled_1x03_Pitch2.54mm" H 3800 2000 50  0001 C CNN
+F 3 "" H 3800 2000 50  0001 C CNN
+	1    3800 2000
+	1    0    0    -1
+$EndComp
+$Comp
+L GND #PWR012
+U 1 1 5B394187
+P 3050 1750
+F 0 "#PWR012" H 3050 1500 50  0001 C CNN
+F 1 "GND" H 3050 1600 50  0000 C CNN
+F 2 "" H 3050 1750 50  0001 C CNN
+F 3 "" H 3050 1750 50  0001 C CNN
+	1    3050 1750
+	1    0    0    -1
+$EndComp
+$Comp
+L VCC #PWR013
+U 1 1 5B3941B7
+P 2850 1850
+F 0 "#PWR013" H 2850 1700 50  0001 C CNN
+F 1 "VCC" H 2850 2000 50  0000 C CNN
+F 2 "" H 2850 1850 50  0001 C CNN
+F 3 "" H 2850 1850 50  0001 C CNN
+	1    2850 1850
+	1    0    0    -1
+$EndComp
+Wire Wire Line
+	2100 3200 2100 3300
+Wire Wire Line
+	1700 3200 1700 3300
+Wire Wire Line
+	1250 3200 1250 3300
+Wire Wire Line
+	6000 2600 6400 2600
+Wire Wire Line
+	7200 3000 7200 3150
+Wire Wire Line
+	6000 3100 7200 3100
+Wire Wire Line
+	2100 3600 2100 3750
+Wire Wire Line
+	1700 3600 1700 3750
+Wire Wire Line
+	1250 3600 1250 3750
+Wire Wire Line
+	2500 4850 2500 5400
+Wire Wire Line
+	2500 3550 2500 3650
+Wire Wire Line
+	2500 4050 2500 4550
+Connection ~ 2500 4250
+Wire Wire Line
+	1850 4700 1850 4850
+Wire Wire Line
+	1300 4700 1300 4850
+Wire Wire Line
+	6850 3700 3300 3700
+Wire Wire Line
+	3300 3700 3300 3100
+Wire Wire Line
+	6850 3800 3200 3800
+Wire Wire Line
+	6850 3900 3100 3900
+Connection ~ 3100 2700
+Wire Wire Line
+	6850 4000 3000 4000
+Connection ~ 3000 2800
+Wire Wire Line
+	6850 3600 6700 3600
+Wire Wire Line
+	6850 4100 6050 4100
+Wire Wire Line
+	6700 3600 6700 3100
+Connection ~ 6700 3100
+Wire Wire Line
+	6050 4100 6050 2600
+Connection ~ 6050 2600
 Wire Wire Line
 	3000 4000 3000 2800
@@
 Wire Wire Line
 	2850 4250 2500 4250
+Wire Wire Line
+	3300 3000 3300 2100
+Wire Wire Line
+	3300 2100 3600 2100
+Wire Wire Line
+	3600 2000 2850 2000
+Wire Wire Line
+	2850 2000 2850 1850
+Wire Wire Line
+	3600 1900 3600 1750
+Wire Wire Line
+	3600 1750 3050 1750
+Wire Wire Line
+	7200 2600 7200 2700
+Wire Wire Line
+	7200 2600 7000 2600
+Connection ~ 7200 3100
+Wire Wire Line
+	6250 2450 6250 2600
+Connection ~ 6250 2600
 $EndSCHEMATC
