File: boardAttinyReflexos/attinyReflexos.sch (KiCad schematic (older format))
At the start: 13 parts, among them J1 Conn_01x06_Female, J2 Conn_01x03_Female, SW1 SW_DPST_x2, SW2 SW_DIP_x01, U1 ATTINY85-20PU

Commit message: better readme
Parts:
- BT1: symbol Battery_Cell -> attinyReflexos-rescue:Battery_Cell
- D1, D2, D3: symbol LED -> attinyReflexos-rescue:LED
- J1: symbol Conn_01x06_Female -> attinyReflexos-rescue:Conn_01x06_Female
- J2: symbol Conn_01x03_Female -> attinyReflexos-rescue:Conn_01x03_Female
- R1, R2, R3, R4: symbol R -> attinyReflexos-rescue:R
- SW1: symbol SW_DPST_x2 -> attinyReflexos-rescue:SW_DPST_x2
- SW2: footprint myfootprint:switchSlide -> (none); symbol SW_DIP_x01 -> attinyReflexos-rescue:SW_DIP_x01
- U1: symbol ATTINY85-20PU -> attinyReflexos-rescue:ATTINY85-20PU
Changed lines of the file:
@@
-EESchema Schematic File Version 2
-LIBS:power
-LIBS:device
-LIBS:switches
-LIBS:relays
-LIBS:motors
-LIBS:transistors
-LIBS:conn
-LIBS:linear
-LIBS:regul
-LIBS:74xx
-LIBS:cmos4000
-LIBS:adc-dac
-LIBS:memory
-LIBS:xilinx
-LIBS:microcontrollers
-LIBS:dsp
-LIBS:microchip
-LIBS:analog_switches
-LIBS:motorola
-LIBS:texas
-LIBS:intel
-LIBS:audio
-LIBS:interface
-LIBS:digital-audio
-LIBS:philips
-LIBS:display
-LIBS:cypress
-LIBS:siliconi
-LIBS:opto
-LIBS:atmel
-LIBS:contrib
-LIBS:valves
+EESchema Schematic File Version 4
 LIBS:attinyReflexos-cache
-EELAYER 25 0
+EELAYER 26 0
 EELAYER END
 $Descr A4 11693 8268
@@
 $EndDescr
 $Comp
-L ATTINY85-20PU U1
+L attinyReflexos-rescue:ATTINY85-20PU U1
 U 1 1 59CAB53C
 P 4650 2850
@@
 $EndComp
 $Comp
-L R R3
+L attinyReflexos-rescue:R R3
 U 1 1 59CAB571
 P 1700 3050
@@
 $EndComp
 $Comp
-L R R4
+L attinyReflexos-rescue:R R4
 U 1 1 59CAB662
 P 2100 3050
@@
 $EndComp
 $Comp
-L R R2
+L attinyReflexos-rescue:R R2
 U 1 1 59CAB6B1
 P 1250 3050
@@
 $EndComp
 $Comp
-L LED D2
+L attinyReflexos-rescue:LED D2
 U 1 1 59CAB6CC
 P 1700 3450
@@
 $EndComp
 $Comp
-L LED D1
+L attinyReflexos-rescue:LED D1
 U 1 1 59CAB7D2
 P 1250 3450
@@
 $EndComp
 $Comp
-L LED D3
+L attinyReflexos-rescue:LED D3
 U 1 1 59CAB7FE
 P 2100 3450
@@
 $EndComp
 $Comp
-L SW_DPST_x2 SW1
+L attinyReflexos-rescue:SW_DPST_x2 SW1
 U 1 1 59CAB9A7
 P 2500 3850
@@
 $EndComp
 $Comp
-L Battery_Cell BT1
+L attinyReflexos-rescue:Battery_Cell BT1
 U 1 1 59D92230
 P 7200 2900
@@
 $EndComp
 $Comp
-L GND #PWR01
+L power:GND #PWR01
 U 1 1 5A74B21D
 P 1250 3750
@@
 $EndComp
 $Comp
-L R R1
+L attinyReflexos-rescue:R R1
 U 1 1 5A74B427
 P 2500 4700
@@
 $EndComp
 $Comp
-L VCC #PWR02
+L power:VCC #PWR02
 U 1 1 5A74B55B
 P 2500 3550
@@
 $EndComp
 $Comp
-L GND #PWR03
+L power:GND #PWR03
 U 1 1 5A74B1B1
 P 2100 3750
@@
 $EndComp
 $Comp
-L GND #PWR04
+L power:GND #PWR04
 U 1 1 5A74B1E4
 P 1700 3750
@@
 $EndComp
 $Comp
-L GND #PWR05
+L power:GND #PWR05
 U 1 1 5A74B35F
 P 2500 5400
@@
 $EndComp
 $Comp
-L VCC #PWR06
+L power:VCC #PWR06
 U 1 1 5A74BBC2
 P 6250 2450
@@
 $EndComp
 $Comp
-L GND #PWR07
+L power:GND #PWR07
 U 1 1 5A74BC27
 P 7200 3150
@@
 $EndComp
 $Comp
-L PWR_FLAG #FLG08
+L power:PWR_FLAG #FLG08
 U 1 1 5A74BF8B
 P 1300 4700
@@
 $EndComp
 $Comp
-L PWR_FLAG #FLG09
+L power:PWR_FLAG #FLG09
 U 1 1 5A74BFFF
 P 1850 4850
@@
 $EndComp
 $Comp
-L GND #PWR010
+L power:GND #PWR010
 U 1 1 5A74C035
 P 1300 4850
@@
 $EndComp
 $Comp
-L VCC #PWR011
+L power:VCC #PWR011
 U 1 1 5A74C064
 P 1850 4700
@@
 $EndComp
 $Comp
-L Conn_01x06_Female J1
+L attinyReflexos-rescue:Conn_01x06_Female J1
 U 1 1 5B04506B
 P 7050 3800
@@
 $EndComp
 $Comp
-L SW_DIP_x01 SW2
+L attinyReflexos-rescue:SW_DIP_x01 SW2
 U 1 1 5B048E78
 P 6700 2600
 F 0 "SW2" H 6700 2750 50  0000 C CNN
 F 1 "SW_DIP_x01" H 6700 2450 50  0000 C CNN
-F 2 "myfootprint:switchSlide" H 6700 2600 50  0001 C CNN
+F 2 "" H 6700 2600 50  0001 C CNN
 F 3 "" H 6700 2600 50  0001 C CNN
 	1    6700 2600
@@
 $EndComp
 $Comp
-L Conn_01x03_Female J2
+L attinyReflexos-rescue:Conn_01x03_Female J2
 U 1 1 5B393E6D
 P 3800 2000
@@
 $EndComp
 $Comp
-L GND #PWR012
+L power:GND #PWR012
 U 1 1 5B394187
 P 3050 1750
@@
 $EndComp
 $Comp
-L VCC #PWR013
+L power:VCC #PWR013
 U 1 1 5B3941B7
 P 2850 1850
@@
 	1250 3200 1250 3300
 Wire Wire Line
-	6000 2600 6400 2600
-Wire Wire Line
-	7200 3000 7200 3150
-Wire Wire Line
-	6000 3100 7200 3100
+	6000 2600 6050 2600
+Wire Wire Line
+	7200 3000 7200 3100
+Wire Wire Line
+	6000 3100 6700 3100
 Wire Wire Line
 	2100 3600 2100 3750
@@
 	2500 3550 2500 3650
 Wire Wire Line
-	2500 4050 2500 4550
+	2500 4050 2500 4250
 Connection ~ 2500 4250
 Wire Wire Line
@@
 Connection ~ 3200 2600
 Wire Wire Line
-	1250 2600 3300 2600
-Wire Wire Line
-	1700 2700 3300 2700
-Wire Wire Line
-	2100 2800 3300 2800
+	1250 2600 3200 2600
+Wire Wire Line
+	1700 2700 3100 2700
+Wire Wire Line
+	2100 2800 3000 2800
 Wire Wire Line
 	1250 2600 1250 2900
@@
 	6250 2450 6250 2600
 Connection ~ 6250 2600
+Wire Wire Line
+	2500 4250 2500 4550
+Wire Wire Line
+	3100 2700 3300 2700
+Wire Wire Line
+	3000 2800 3300 2800
+Wire Wire Line
+	6700 3100 7200 3100
+Wire Wire Line
+	6050 2600 6250 2600
+Wire Wire Line
+	3200 2600 3300 2600
+Wire Wire Line
+	7200 3100 7200 3150
+Wire Wire Line
+	6250 2600 6400 2600
 $EndSCHEMATC

Commit message: caixa en openscad
Parts:
- SW2: footprint (none) -> myfootprint:sk12d07v
Changed lines of the file:
@@
 F 0 "SW2" H 6700 2750 50  0000 C CNN
 F 1 "SW_DIP_x01" H 6700 2450 50  0000 C CNN
-F 2 "" H 6700 2600 50  0001 C CNN
+F 2 "myfootprint:sk12d07v" H 6700 2600 50  0001 C CNN
 F 3 "" H 6700 2600 50  0001 C CNN
 	1    6700 2600
